File: a-side/a-side.kicad_pcb (KiCad board)
At the start: 2 copper layers, 95 x 60 mm, 18 parts, among them IC1 GL3510-OSY52, IC2 GL823K, IC3 GL823K, J1 503500-0993, J2 503500-0993, J3 USB_A, J4 USB_C_Receptacle, Y1 Crystal

Commit message: oops
accidentally left out a few files whoops
Parts:
- removed IC3: GL823K, Package_SO:SOIC-16_3.9x9.9mm_P1.27mm
- added C10: 22pF, Capacitor_SMD:C_0805_2012Metric, F.Cu at (57.5, 109.3)
- added C11: 22pF, Capacitor_SMD:C_0805_2012Metric, F.Cu at (57.5, 112.3)
- added C12: 100nF, Capacitor_SMD:C_0805_2012Metric, F.Cu at (57.5, 115.3)
- added C13: 100nF, Capacitor_SMD:C_0805_2012Metric, F.Cu at (62.0, 100.2)
- added C14: 100nF, Capacitor_SMD:C_0805_2012Metric, F.Cu at (62.0, 103.2)
- added C15: 100nF, Capacitor_SMD:C_0805_2012Metric, F.Cu at (62.0, 106.3)
- added C16: 100nF, Capacitor_SMD:C_0805_2012Metric, F.Cu at (62.0, 109.3)
- added C17: 100nF, Capacitor_SMD:C_0805_2012Metric, F.Cu at (62.0, 112.3)
- added C18: 0.1uF, Capacitor_SMD:C_0805_2012Metric, F.Cu at (77.6, 123.8)
- added C9: 100nF, Capacitor_SMD:C_0805_2012Metric, F.Cu at (57.5, 106.3)
- added GL850G1: GL850G, GL850G Model:28SSOP, F.Cu at (69.6, 120.6)
- added J5: USB_A, Connector_USB:USB_A_Molex_67643_Horizontal, F.Cu at (56.5, 84.7)
- added R3: 10kR, Resistor_SMD:R_0805_2012Metric, F.Cu at (71.3, 71.5)
- added R4: 680R, Resistor_SMD:R_0805_2012Metric, F.Cu at (71.3, 74.4)
- added R5: 100kohm, Resistor_SMD:R_0805_2012Metric, F.Cu at (71.3, 77.4)
- added R6: 100kR, Resistor_SMD:R_0805_2012Metric, F.Cu at (71.3, 80.3)
- added R7: 5.1kR, Resistor_SMD:R_0805_2012Metric, F.Cu at (71.3, 83.3)
- added R8: 5.1kR, Resistor_SMD:R_0805_2012Metric, F.Cu at (71.3, 86.2)
- added U1: AMS1117CD-3.3, Package_TO_SOT_SMD:TO-252-3_TabPin2, F.Cu at (57.8, 121.0)
- added U2: SRV05-4, Package_TO_SOT_SMD:SOT-23-6, F.Cu at (78.0, 120.1)
- C1: value C -> 10uF; footprint Capacitor_SMD:C_0603_1608Metric -> Capacitor_SMD:C_0805_2012Metric
- C2: value C -> 22uF; footprint Capacitor_SMD:C_0603_1608Metric -> Capacitor_SMD:C_0805_2012Metric
- C3: footprint Capacitor_SMD:C_0603_1608Metric -> Capacitor_SMD:C_0805_2012Metric
- C4, C5, C6, C7, C8: value 0.1uF -> 100nF; footprint Capacitor_SMD:C_0603_1608Metric -> Capacitor_SMD:C_0805_2012Metric
- IC1: value GL3510-OSY52 -> GL823K; footprint gl3510:QFN40P800X800X80-65N-D -> GL823K Model by Genesys Logic:SOP64P600X175-16N
- IC2: footprint Package_SO:SOIC-16_3.9x9.9mm_P1.27mm -> GL823K Model by Genesys Logic:SOP64P600X175-16N
- J1: value 503500-0993 -> Conn_01x06; footprint 5035000993:5035000993 -> Connector_PinHeader_2.54mm:PinHeader_1x06_P2.54mm_Vertical
- J3: value USB_A -> 503500-0993; footprint Connector_USB:USB_A_CNCTech_1001-011-01101_Horizontal -> 5035000993:5035000993
- J4: value USB_C_Receptacle -> USB_A; footprint Connector_USB:USB_C_Receptacle_Molex_105450-0101 -> Connector_USB:USB_A_Molex_67643_Horizontal
- R1: value 10k -> 100kR; footprint Resistor_SMD:R_0603_1608Metric -> Resistor_SMD:R_0805_2012Metric
- R2: value 20k -> 100kR; footprint Resistor_SMD:R_0603_1608Metric -> Resistor_SMD:R_0805_2012Metric
- Y1: footprint Crystal:Crystal_SMD_5032-2Pin_5.0x3.2mm -> Crystal:Crystal_SMD_3225-4Pin_3.2x2.5mm_HandSoldering
- moved J1 139.9 mm to (66.5, 101.0)
- moved C1 137.9 mm to (53.1, 100.2)
- moved C3 137.9 mm to (53.1, 106.3)
- moved C2 137.8 mm to (53.1, 103.2)
- moved C6 133.6 mm to (53.1, 115.3), turned to 0 degrees
- moved C4 133.4 mm to (53.1, 109.3)
- moved C8 123.6 mm to (57.5, 103.2)
- moved C7 122.9 mm to (57.5, 100.2), turned to 0 degrees
- moved C5 122.0 mm to (53.1, 112.3)
- moved Y1 118.6 mm to (71.7, 90.0)
- moved R1 109.9 mm to (71.3, 65.6), turned to 0 degrees
- moved IC1 109.0 mm to (73.0, 102.1)
- moved R2 104.3 mm to (71.3, 68.5), turned to 0 degrees
- moved IC2 93.9 mm to (73.0, 108.7)
- moved J4 85.6 mm to (56.5, 67.4), turned to 0 degrees
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Connections:
- C1 pad 1: Net-(IC1-X1) -> VBUS
- C1 pad 2: GND -> Net-(C1-Pad2)
- C2 pad 1: Net-(IC1-X2) -> +3.3V
- C2 pad 2: GND -> Net-(C18-Pad2)
- C3 pad 1: GND -> Net-(C1-Pad2)
- C3 pad 2: +3.3V -> GND
- C4 pad 1: GND -> +3.3V
- C4 pad 2: +3.3V -> GND
- C5 pad 1: GND -> VBUS
- C5 pad 2: +3.3V -> GND
- C6 pad 1: GND -> +3.3V
- C6 pad 2: +3.3V -> GND
- C7 pad 1: GND -> +3.3V
- C7 pad 2: +3.3V -> GND
- C8 pad 1: GND -> +3.3V
- C8 pad 2: +3.3V -> GND
- IC1 pad 1: unconnected-(IC1-TXN1_P3-Pad1) -> GND
- IC1 pad 10: unconnected-(IC1-DM_P4-Pad10) -> VBUS
- IC1 pad 13: unconnected-(IC1-VP12_P4-Pad13) -> Net-(IC1-VDD)
- IC1 pad 14: unconnected-(IC1-RXN1_P4-Pad14) -> GND
- IC1 pad 15: unconnected-(IC1-RXP1_P4-Pad15) -> /SD1_DP
- IC1 pad 16: Net-(IC1-RTERM) -> /SD1_DM
- IC1 pad 2: unconnected-(IC1-TXP1_P3-Pad2) -> /SD1_D1
- IC1 pad 3: unconnected-(IC1-VP12_P3-Pad3) -> /SD1_D0
- IC1 pad 4: unconnected-(IC1-RXN1_P3-Pad4) -> /SD1_CLK
- IC1 pad 5: unconnected-(IC1-RXP1_P3-Pad5) -> /SD1_CMD
- IC1 pad 6: unconnected-(IC1-DP_P3-Pad6) -> /SD1_D3
- IC1 pad 7: unconnected-(IC1-DM_P3-Pad7) -> /SD1_D2
- IC1 pad 8: +3.3V -> /SD1_PWR
- IC1 pad 9: unconnected-(IC1-DP_P4-Pad9) -> Net-(IC1-VDD)
- IC2 pad 10: unconnected-(IC2-5V-Pad10) -> VBUS
- IC2 pad 13: +3.3V -> Net-(IC2-VDD)
- IC2 pad 15: /DP -> /SD2_DP
- IC2 pad 16: /DM -> /SD2_DM
- IC2 pad 2: /D1 -> /SD2_D1
- IC2 pad 3: unconnected-(IC2-D0-Pad3) -> /SD2_D0
- IC2 pad 4: /CLK -> /SD2_CLK
- IC2 pad 5: /CMD -> /SD2_CMD
- IC2 pad 6: unconnected-(IC2-D3-Pad6) -> /SD2_D3
- IC2 pad 7: /D2 -> /SD2_D2
- IC2 pad 8: unconnected-(IC2-PMOS-Pad8) -> /SD2_PWR
- IC2 pad 9: +3.3V -> Net-(IC2-VDD)
- J1 pad 1: unconnected-(J1-Pad1) -> VBUS
- J1 pad 2: unconnected-(J1-Pad2) -> GND
- J1 pad 3: unconnected-(J1-Pad3) -> /USB_DP
- J1 pad 4: unconnected-(J1-Pad4) -> /USB_DM
- J1 pad 5: unconnected-(J1-Pad5) -> Net-(J1-Pin_5)
- J1 pad 6: unconnected-(J1-Pad6) -> Net-(J1-Pin_6)
- J2 pad 5: unconnected-(J2-Pad5) -> /SD1_CLK
- J2 pad 6: unconnected-(J2-Pad6) -> GND
- J2 pad 7: unconnected-(J2-Pad7) -> /SD1_D0
- J2 pad 8: unconnected-(J2-Pad8) -> /SD1_D1
- J2 pad 9: unconnected-(J2-Pad9) -> GND
- J2 pad D1: /D1 -> unconnected-(J2-CARD_DETECT_1-PadD1)
- J2 pad D2: /D2 -> unconnected-(J2-CARD_DETECT_2-PadD2)
- J2 pad MP1: /CMD -> /SD1_D2
- J2 pad MP2: /CLK -> /SD1_D3
- J2 pad MP3: +3.3V -> /SD1_CMD
- J2 pad MP4: GND -> /SD1_PWR
- J3 pad 4: GND -> unconnected-(J3-Pad4)
- J3 pad 5: unconnected-(J3-Shield-Pad5) -> /SD2_CLK
- R1 pad 1: Net-(IC1-RESETJ) -> Net-(GL850G1-PSELF)
- R1 pad 2: Net-(IC1-VBUS) -> GND
- R2 pad 1: Net-(IC1-RTERM) -> Net-(GL850G1-PGANG)
- R2 pad 2: GND -> +3V3
- Y1 pad 1: Net-(IC1-X2) -> Net-(GL850G1-X1)
- Y1 pad 2: Net-(IC1-X1) -> Net-(GL850G1-X2)
