File: a-side/a-side.kicad_pcb (KiCad board)
At the start: 2 copper layers, 95 x 60 mm, 41 parts, among them IC1 GL823K, IC2 GL823K, J1 Conn_01x04, J2 503500-0993, J3 503500-0993, J4 USB_A, J5 USB_A, U1 AMS1117CD-3.3, U2 SRV05-4, Y1 Crystal

Commit message: sorrryyy
this is a commit from last night, started layout, fixed schematic issues and well. ready to fix problems now
Parts:
- removed the R7 at (71.3, 83.3)
- removed the R8 at (71.3, 86.2)
- moved D2 146.8 mm to (165.8, 122.8)
- moved R8 138.9 mm to (166.5, 84.5)
- moved J1 125.2 mm to (172.2, 71.0)
- moved C3 121.1 mm to (168.3, 69.0)
- moved C1 115.5 mm to (164.3, 69.0)
- moved C2 115.2 mm to (164.3, 73.0)
- moved J3 112.8 mm to (156.3, 95.2)
- moved D1 112.3 mm to (129.0, 122.5)
- moved U1 108.6 mm to (155.3, 73.2), turned to 180 degrees
- moved C18 103.9 mm to (168.3, 73.0)
- moved U2 98.9 mm to (167.6, 78.5)
- moved C17 97.4 mm to (155.8, 85.8)
- moved C16 94.4 mm to (155.0, 93.0)
- moved C15 94.3 mm to (155.0, 91.0), turned to 180 degrees
- moved R7 89.1 mm to (116.8, 88.2)
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Routing:
- net VBUS: track 0.00 -> 66.9 mm, vias 0 -> 1
- net /USBA2_DP: track 0.00 -> 65.2 mm
- net /USB_DM: track 0.00 -> 64.2 mm, vias 0 -> 2
- net /USB_DP: track 0.00 -> 62.4 mm, vias 0 -> 2
- net /USBA2_DM: track 0.00 -> 57.6 mm
- net +3.3V: track 0.00 -> 55.4 mm
- net Net-(D1-K): track 0.00 -> 44.6 mm, vias 0 -> 2
- net Net-(D2-K): track 0.00 -> 39.4 mm
- net /USBA1_DM: track 0.00 -> 38.0 mm
- net /USBA1_DP: track 0.00 -> 38.0 mm, vias 0 -> 2
- net /SD2_D2: track 0.00 -> 34.4 mm
- net /SD1_D2: track 0.00 -> 34.4 mm
- net /SD2_DM: track 0.00 -> 34.2 mm, vias 0 -> 2
- net /SD2_DP: track 0.00 -> 33.5 mm
- net Net-(IC1-VDD): track 0.00 -> 28.4 mm
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- added copper zone on B.Cu, net GND
- added copper zone on F.Cu, net GND
Other:
- board text added: "gonna be switching between schematic and editor a lot, NOT AFK!!"
