File: a-side/a-side.kicad_pcb (KiCad board)
At the start: 2 copper layers, 95 x 60 mm, 39 parts, among them IC1 GL823K, IC2 GL823K, J2 USB_C_Receptacle_USB2.0_14P, J4 USB_A, J5 USB_A, J6 SD_Card_Receptacle, J7 SD_Card_Receptacle, U1 AMS1117CD-3.3, U2 SRV05-4, Y1 Crystal

Commit message: small worksesh
finishweed my test earlier decided to get some work (NOT) done. scoured the internet for a footprint and i think i found one chat, gonna add it after studying
Parts:
- added C19: 100nF, Capacitor_SMD:C_0805_2012Metric, F.Cu at (65.5, 52.5)
- added R10: 5.1k, Resistor_SMD:R_0805_2012Metric, F.Cu at (74.3, 52.2)
- added R9: 5.1k, Resistor_SMD:R_0805_2012Metric, F.Cu at (74.3, 49.3)
- J6, J7: footprint Connector_Card:SD_TE_2041021 -> Connector_Card:SD_Card_Device_16mm_SlotDepth
- moved J7 149.3 mm to (41.3, 39.3)
- moved J2 142.5 mm to (34.2, 53.8), turned to 0 degrees
- moved J6 142.5 mm to (41.3, 21.3)
- moved D2 134.9 mm to (49.6, 54.1)
- moved U2 132.2 mm to (43.1, 57.7)
- moved U1 123.4 mm to (35.3, 44.5), turned to 0 degrees
- moved C3 113.9 mm to (56.6, 46.5)
- moved C2 111.7 mm to (56.6, 43.5)
- moved C1 111.4 mm to (56.6, 40.5)
- moved D1 106.8 mm to (49.6, 51.1)
- moved C18 105.5 mm to (65.5, 49.5)
- moved IC2 103.9 mm to (76.8, 14.4)
- moved C16 102.9 mm to (65.5, 43.5)
- moved C15 102.8 mm to (65.5, 40.5), turned to 0 degrees
- moved C17 98.4 mm to (65.5, 46.5)
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Connections:
- IC1 pad 8: /SD1_PWR -> unconnected-(IC1-PMOS-Pad8)
- IC2 pad 8: /SD2_PWR -> unconnected-(IC2-PMOS-Pad8)
- J2 pad A5: unconnected-(J2-CC1-PadA5) -> Net-(J2-CC1)
- J2 pad B5: unconnected-(J2-CC2-PadB5) -> Net-(J2-CC2)
- J6 pad 4: /SD1_PWR -> +3.3V
- J7 pad 4: /SD2_PWR -> +3.3V
- U2 pad 5: unconnected-(U2-VP-Pad5) -> VBUS
Routing:
- net +3.3V: track 58.9 -> 0.00 mm
- net /USBA2_DM: track 47.1 -> 0.00 mm
- net VBUS: track 47.0 -> 0.00 mm
- net /USBA2_DP: track 42.8 -> 0.00 mm
- net Net-(D1-K): track 41.1 -> 0.00 mm
- net Net-(D2-K): track 36.7 -> 0.00 mm
- net /SD2_DP: track 35.6 -> 0.00 mm
- net /SD2_DM: track 32.7 -> 0.00 mm
- net Net-(GL850G1-~{OVCUR2}): track 24.3 -> 0.00 mm
- net Net-(GL850G1-~{OVCUR1}): track 17.8 -> 0.00 mm
- net Net-(IC1-VDD): track 15.3 -> 0.00 mm
- net Net-(IC2-VDD): track 14.9 -> 0.00 mm
- net /USB_DM: track 13.7 -> 0.00 mm
- net Net-(GL850G1-X1): track 13.6 -> 0.00 mm
- net /USB_DP: track 11.5 -> 0.00 mm
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Other:
- board size 95 x 60 mm -> 95 x 55 mm
- board text removed: "I don't think the footprints are right."
- board text removed: "These two are RISKY!"
- board text removed: "gonna be switching between schematic and editor a lot, NOT AFK!!"
