File: a-side/a-side.kicad_sch (KiCad schematic)
At the start: 19 parts, among them IC1 GL3510-OSY52, IC2 GL823K, IC3 GL823K, J1 503500-0993, J2 503500-0993, J3 USB_A, J4 USB_C_Receptacle, P1 USB_C_Plug, Y1 Crystal

Commit message: oops cant forget to commit!
soo mostly just about finished my pcb schema? waiting on some of the errors to fix themselves (jk, ill do it tmrw) and assigning footprints tonight and ill do 1 more commit in a bit :)
Parts:
- removed IC1: GL3510-OSY52, gl3510:QFN40P800X800X80-65N-D, symbol GL3510-OSY52:GL3510-OSY52
- removed IC3: GL823K, Package_SO:SOIC-16_3.9x9.9mm_P1.27mm, symbol GL823K:GL823K
- removed J1: 503500-0993, 5035000993:5035000993, symbol 503500-0993:503500-0993
- removed J3: USB_A, Connector_USB:USB_A_CNCTech_1001-011-01101_Horizontal, symbol Connector:USB_A
- removed J4: USB_C_Receptacle, Connector_USB:USB_C_Receptacle_Molex_105450-0101, symbol Connector:USB_C_Receptacle
- removed P1: USB_C_Plug, symbol Connector:USB_C_Plug
- added C10, C11: 22pF, Capacitor_SMD:C_0805_2012Metric, symbol Device:C
- added C12, C13, C14, C15, C16, C17, C9: 100nF, Capacitor_SMD:C_0805_2012Metric, symbol Device:C
- added GL850G1: GL850G, GL850G:28SSOP, symbol GL850G:GL850G
- added IC1: GL823K, GL823K:SOP64P600X175-16N, symbol GL823K:GL823K
- added J1: USB_C_Receptacle, Connector_USB:USB_C_Receptacle_HRO_TYPE-C-31-M-12, symbol Connector:USB_C_Receptacle
- added J3: 503500-0993, symbol 503500-0993:503500-0993
- added J4, J5: USB_A, Connector_USB:USB_A_Molex_67643_Horizontal, symbol Connector:USB_A
- added R3: 10kR, Resistor_SMD:R_0805_2012Metric, symbol Device:R
- added R4: 680ohm, Resistor_SMD:R_0805_2012Metric, symbol Device:R
- added R5: 100kohm, Resistor_SMD:R_0805_2012Metric, symbol Device:R
- added R6: 100kR, Resistor_SMD:R_0805_2012Metric, symbol Device:R
- added R7, R8: 5.1k, Resistor_SMD:R_0805_2012Metric, symbol Device:R
- added U1: AMS1117CD-3.3, Package_TO_SOT_SMD:TO-252-3_TabPin2, symbol Regulator_Linear:AMS1117CD-3.3
- C1, C2: value C -> 10uF; footprint Capacitor_SMD:C_0603_1608Metric -> Capacitor_SMD:C_0805_2012Metric
- C3, C4, C5, C6, C7, C8: value 0.1uF -> 100nF; footprint Capacitor_SMD:C_0603_1608Metric -> Capacitor_SMD:C_0805_2012Metric
- IC2: footprint Package_SO:SOIC-16_3.9x9.9mm_P1.27mm -> GL823K:SOP64P600X175-16N
- J2: footprint 5035000993:5035000993 -> (none)
- R1: value 10k -> 100kR; footprint Resistor_SMD:R_0603_1608Metric -> Resistor_SMD:R_0805_2012Metric
- R2: value 20k -> 100kR; footprint Resistor_SMD:R_0603_1608Metric -> Resistor_SMD:R_0805_2012Metric
- Y1: footprint Crystal:Crystal_SMD_5032-2Pin_5.0x3.2mm -> Crystal:Crystal_SMD_3225-4Pin_3.2x2.5mm
Connections:
- net +3.3V: now also C2.1, C3.1, C4.1, C6.1, C7.1, C8.1, C9.1, GL850G1.1 (AVDD@1), GL850G1.10 (AVDD@3), GL850G1.16 (DVDD), GL850G1.24 (3V3), GL850G1.5 (AVDD@2), U1.2 (VO); no longer C3.2, C4.2, C5.2, C6.2, C7.2, C8.2, IC2.13 (VDDA), IC2.9 (VDD), J2.MP3
- net GND: now also C3.2, C4.2, C5.2, C6.2, C7.2, C8.2, J2.6, J2.9, R1.2, C10.1, C11.2, C12.2, C13.1, C14.2, C15.1, C16.2, C17.2, C9.2, GL850G1.14 (TEST), GL850G1.15 (GND), IC1.1 (VSS_1), IC1.14 (VSS_2), J1.A1 (GND), J1.A12 (GND), J1.B1 (GND), J1.B12 (GND), J1.S1 (SHIELD), J3.6, J3.9, J4.4 (GND), J4.5 (Shield), J5.4 (GND), J5.5 (Shield), R4.2, R7.2, R8.1, U1.1 (GND); no longer C3.1, C4.1, C5.1, C6.1, C7.1, C8.1, J2.MP4, R2.2
- net at R2.1: now also GL850G1.18 (PGANG)
- net at R1.1: now also GL850G1.17 (PSELF)
- net at Y1.1: now also C10.2, GL850G1.6 (X1); no longer C2.1
- net at Y1.2: now also C11.1, GL850G1.7 (X2); no longer C1.1
- net SD1_CLK: now reaches J2.5
- net SD1_CLK: now also IC1.4 (CLK)
- net SD1_D0: now reaches J2.7
- net SD1_D0: now also IC1.3 (D0)
- net SD1_D1: now reaches J2.8
- net SD1_D1: now also IC1.2 (D1)
- net VBUS: now reaches IC2.10 (5V)
- net VBUS: now also C1.1, C5.1, C13.2, C15.2, GL850G1.23 (5V), IC1.10 (5V), J1.A4 (VBUS), J1.A9 (VBUS), J1.B4 (VBUS), J1.B9 (VBUS), J4.1 (VBUS), J5.1 (VBUS), U1.3 (VI)
- net SD2_D0: now reaches IC2.3 (D0)
- net SD2_D0: now also J3.7
- net SD2_D3: now reaches IC2.6 (D3)
- net SD2_D3: now also J3.MP2
- net SD2_PWR: now reaches IC2.8 (PMOS)
- net SD2_PWR: now also J3.MP4
- net CLK renamed SD1_D3
- net SD1_D3: now also IC1.6 (D3); no longer IC2.4 (CLK)
- net CMD renamed SD1_D2
- net SD1_D2: now also IC1.7 (D2); no longer IC2.5 (CMD)
- net D1: no longer names the net of J2.D1 (CARD_DETECT_1)
- net D1: no longer IC2.2 (D1)
- net D2: no longer names the net of J2.D2 (CARD_DETECT_2)
- net D2: no longer IC2.7 (D2)
- net DM renamed SD2_DM
- net SD2_DM: now also GL850G1.2 (DM2)
- net DP renamed SD2_DP
- net SD2_DP: now also GL850G1.3 (DP2)
- new net: J1.A5 (CC1), R7.1
- new net: GL850G1.19 (~{OVCUR2}), R6.1
- new net: GL850G1.4 (RREF), R4.1
- new net: C17.1, IC2.13 (VDDA)
- new net: C16.1, IC2.9 (VDD)
- new net: C12.1, IC1.9 (VDD)
- new net: J1.B5 (CC2), R8.2
- new net: C14.1, IC1.13 (VDDA)
- new net: GL850G1.13 (~{RESET}), R3.1
- new net: GL850G1.21 (~{OVCUR1}), R5.1
- new net +3V3: R2.2, R3.2, R5.2, R6.2
- new net SD1_CMD: IC1.5 (CMD), J2.MP3
- new net SD1_DM: GL850G1.27 (DM1), IC1.16 (DM)
- new net SD1_DP: GL850G1.28 (DP1), IC1.15 (DP)
- new net SD1_PWR: IC1.8 (PMOS), J2.MP4
- new net SD2_CLK: IC2.4 (CLK), J3.5
- new net SD2_CMD: IC2.5 (CMD), J3.MP3
- new net SD2_D1: IC2.2 (D1), J3.8
- new net SD2_D2: IC2.7 (D2), J3.MP1
- new net USBA1_DM: GL850G1.8 (DM3), J4.2 (D-)
- new net USBA1_DP: GL850G1.9 (DP3), J4.3 (D+)
- new net USBA2_DM: GL850G1.11 (DM4), J5.2 (D-)
- new net USBA2_DP: GL850G1.12 (DP4), J5.3 (D+)
- new net USB_DM: GL850G1.25 (DM0), J1.A7 (D-), J1.B7 (D-)
- new net USB_DP: GL850G1.26 (DP0), J1.A6 (D+), J1.B6 (D+)
- no-connect marks 4 -> 32
Other:
- note added: "GO DOWN ⬇︎ FOR SD CARD STUFF!!! SORRY!!! I RAN OUT OF SPACE"
- note added: "footprint time! not afk, sorry, this is gonna be really quick i promise"

Commit message: schema done! (kinda)
gonna start fixing erors tomorrow and layout tmrw but yay shcema is 99% mostly kinda done! yay! yay! yay!!! 😸
Parts:
- removed J1: USB_C_Receptacle, Connector_USB:USB_C_Receptacle_HRO_TYPE-C-31-M-12, symbol Connector:USB_C_Receptacle
- added C18: 0.1uF, Capacitor_SMD:C_0805_2012Metric, symbol Device:C
- added J1: Conn_01x06, Connector_PinHeader_2.54mm:PinHeader_1x06_P2.54mm_Vertical, symbol Connector_Generic:Conn_01x06
- added U2: SRV05-4, Package_TO_SOT_SMD:SOT-23-6, symbol Power_Protection:SRV05-4
- C2: value 10uF -> 22uF
- C3: value 100nF -> 0.1uF
- GL850G1: footprint GL850G:28SSOP -> GL850G Model:28SSOP
- IC1, IC2: footprint GL823K:SOP64P600X175-16N -> GL823K Model by Genesys Logic:SOP64P600X175-16N
- J2, J3: footprint (none) -> 5035000993:5035000993
- R4: value 680ohm -> 680R
- R7, R8: value 5.1k -> 5.1kR
- Y1: footprint Crystal:Crystal_SMD_3225-4Pin_3.2x2.5mm -> Crystal:Crystal_SMD_3225-4Pin_3.2x2.5mm_HandSoldering
Connections:
- net +3.3V: no longer C3.1
- net GND: now also C18.1, J1.2 (Pin_2), U2.2 (VN); no longer C1.2, C2.2, R7.2, R8.1
- net USB_DM: now also J1.4 (Pin_4), U2.3 (IO2)
- net USB_DP: now also J1.3 (Pin_3), U2.1 (IO1)
- net VBUS: now also J1.1 (Pin_1)
- net CC1: now reaches R7.1
- net at C17.1, IC2.13 (VDDA): now also C16.1, IC2.9 (VDD)
- net at C12.1, IC1.9 (VDD): now also C14.1, IC1.13 (VDDA)
- net at R8.2: now also J1.6 (Pin_6)
- new net: C1.2, C3.1
- new net: C18.2, C2.2
- new net: J1.5 (Pin_5), R7.2
- new net CC2: R8.1
- no-connect marks 32 -> 25
Other:
- moved on the sheet: C1, C14, C17, C2, C3

Commit message: oops
accidentally left out a few files whoops
Other:
- note removed: "footprint time! not afk, sorry, this is gonna be really quick i promise"
Changed lines of the file:
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@@
 	(generator_version "9.0")
 	(paper "A4")
-	(text "footprint time! not afk, sorry, this is gonna be really quick i promise\n"
-		(exclude_from_sim no)
-		(at 62.484 -20.828 0)
-		(effects
-			(font
-				(size 1.27 1.27)
-			)
-		)
-	)
 	(text "GO DOWN ⬇︎ FOR SD CARD STUFF!!! SORRY!!! I RAN OUT OF SPACE\n"
 		(exclude_from_sim no)
@@
 	(symbol
 		(lib_id "power:PWR_FLAG")
-		(at 91.44 78.74 0)
+		(at 77.47 83.82 0)
 		(unit 1)
 		(exclude_from_sim no)
@@
 		(fields_autoplaced yes)
 		(property "Reference" "#FLG01"
-			(at 91.44 76.835 0)
+			(at 77.47 81.915 0)
 			(effects
 				(font
@@
 		)
 		(property "Value" "PWR_FLAG"
-			(at 91.44 73.66 0)
+			(at 77.47 78.74 0)
 			(effects
 				(font
@@
 		)
 		(property "Footprint" ""
-			(at 91.44 78.74 0)
+			(at 77.47 83.82 0)
 			(effects
 				(font
@@
 		)
 		(property "Datasheet" "~"
-			(at 91.44 78.74 0)
+			(at 77.47 83.82 0)
 			(effects
 				(font
@@
 		)
 		(property "Description" "Special symbol for telling ERC where power comes from"
-			(at 91.44 78.74 0)
+			(at 77.47 83.82 0)
 			(effects
 				(font
@@
 	(symbol
 		(lib_id "power:VBUS")
-		(at 91.44 78.74 180)
+		(at 77.47 83.82 180)
 		(unit 1)
 		(exclude_from_sim no)
@@
 		(fields_autoplaced yes)
 		(property "Reference" "#PWR063"
-			(at 91.44 74.93 0)
+			(at 77.47 80.01 0)
 			(effects
 				(font
@@
 		)
 		(property "Value" "VBUS"
-			(at 91.44 83.82 0)
+			(at 77.47 88.9 0)
 			(effects
 				(font
@@
 		)
 		(property "Footprint" ""
-			(at 91.44 78.74 0)
+			(at 77.47 83.82 0)
 			(effects
 				(font
@@
 		)
 		(property "Datasheet" ""
-			(at 91.44 78.74 0)
+			(at 77.47 83.82 0)
 			(effects
 				(font
@@
 		)
 		(property "Description" "Power symbol creates a global label with name \"VBUS\""
-			(at 91.44 78.74 0)
+			(at 77.47 83.82 0)
 			(effects
 				(font
@@
 	(symbol
 		(lib_id "power:GND")
-		(at 119.38 78.74 0)
+		(at 105.41 83.82 0)
 		(unit 1)
 		(exclude_from_sim no)
@@
 		(fields_autoplaced yes)
 		(property "Reference" "#PWR065"
-			(at 119.38 85.09 0)
+			(at 105.41 90.17 0)
 			(effects
 				(font
@@
 		)
 		(property "Value" "GND"
-			(at 119.38 83.82 0)
+			(at 105.41 88.9 0)
 			(effects
 				(font
@@
 		)
 		(property "Footprint" ""
-			(at 119.38 78.74 0)
+			(at 105.41 83.82 0)
 			(effects
 				(font
@@
 		)
 		(property "Datasheet" ""
-			(at 119.38 78.74 0)
+			(at 105.41 83.82 0)
 			(effects
 				(font
@@
 		)
 		(property "Description" "Power symbol creates a global label with name \"GND\" , ground"
-			(at 119.38 78.74 0)
+			(at 105.41 83.82 0)
 			(effects
 				(font
@@
 	(symbol
 		(lib_id "power:+3V3")
-		(at 106.68 78.74 180)
+		(at 92.71 83.82 180)
 		(unit 1)
 		(exclude_from_sim no)
@@
 		(fields_autoplaced yes)
 		(property "Reference" "#PWR064"
-			(at 106.68 74.93 0)
+			(at 92.71 80.01 0)
 			(effects
 				(font
@@
 		)
 		(property "Value" "+3V3"
-			(at 106.68 83.82 0)
+			(at 92.71 88.9 0)
 			(effects
 				(font
@@
 		)
 		(property "Footprint" ""
-			(at 106.68 78.74 0)
+			(at 92.71 83.82 0)
 			(effects
 				(font
@@
 		)
 		(property "Datasheet" ""
-			(at 106.68 78.74 0)
+			(at 92.71 83.82 0)
 			(effects
 				(font
@@
 		)
 		(property "Description" "Power symbol creates a global label with name \"+3V3\""
-			(at 106.68 78.74 0)
+			(at 92.71 83.82 0)
 			(effects
 				(font
@@
 	(symbol
 		(lib_id "power:PWR_FLAG")
-		(at 106.68 78.74 0)
+		(at 92.71 83.82 0)
 		(unit 1)
 		(exclude_from_sim no)
@@
 		(fields_autoplaced yes)
 		(property "Reference" "#FLG02"
-			(at 106.68 76.835 0)
+			(at 92.71 81.915 0)
 			(effects
 				(font
@@
 		)
 		(property "Value" "PWR_FLAG"
-			(at 106.68 73.66 0)
+			(at 92.71 78.74 0)
 			(effects
 				(font
@@
 		)
 		(property "Footprint" ""
-			(at 106.68 78.74 0)
+			(at 92.71 83.82 0)
 			(effects
 				(font
@@
 		)
 		(property "Datasheet" "~"
-			(at 106.68 78.74 0)
+			(at 92.71 83.82 0)
 			(effects
 				(font
@@
 		)
 		(property "Description" "Special symbol for telling ERC where power comes from"
-			(at 106.68 78.74 0)
+			(at 92.71 83.82 0)
 			(effects
 				(font
@@
 	(symbol
 		(lib_id "power:PWR_FLAG")
-		(at 119.38 78.74 0)
+		(at 105.41 83.82 0)
 		(unit 1)
 		(exclude_from_sim no)
@@
 		(fields_autoplaced yes)
 		(property "Reference" "#FLG03"
-			(at 119.38 76.835 0)
+			(at 105.41 81.915 0)
 			(effects
 				(font
@@
 		)
 		(property "Value" "PWR_FLAG"
-			(at 119.38 73.66 0)
+			(at 105.41 78.74 0)
 			(effects
 				(font
@@
 		)
 		(property "Footprint" ""
-			(at 119.38 78.74 0)
+			(at 105.41 83.82 0)
 			(effects
 				(font
@@
 		)
 		(property "Datasheet" "~"
-			(at 119.38 78.74 0)
+			(at 105.41 83.82 0)
 			(effects
 				(font
@@
 		)
 		(property "Description" "Special symbol for telling ERC where power comes from"
-			(at 119.38 78.74 0)
+			(at 105.41 83.82 0)
 			(effects
 				(font
