File: a-side/a-side.kicad_sch (KiCad schematic)
At the start: 52 parts, among them IC1 GL823K, IC2 GL823K, J2 USB_C_Receptacle_USB2.0_14P, J4 USB_A, J5 USB_A, J6 SD_Card_Receptacle, J7 SD_Card_Receptacle, U1 AMS1117CD-3.3, U2 SRV05-4, Y1 Crystal

Commit message: yea i WISH something changed
but i dont really think it did
Parts:
- removed C1, C2: 10uF, Capacitor_SMD:C_0805_2012Metric, symbol Device:C
- removed C10, C11: 22pF, Capacitor_SMD:C_0805_2012Metric, symbol Device:C
- removed C18, C3: 0.1uF, Capacitor_SMD:C_0805_2012Metric, symbol Device:C
- removed GL850G1: GL850G, GL850G Model:28SSOP, symbol GL850G:GL850G
- removed IC1, IC2: GL823K, GL823K Model by Genesys Logic:SOP64P600X175-16N, symbol GL823K:GL823K
- removed J2: USB_C_Receptacle_USB2.0_14P, Connector_USB:USB_C_Receptacle_GCT_USB4105-xx-A_16P_TopMnt_Horizontal, symbol Connector:USB_C_Receptacle_USB2.0_14P
- removed J4, J5: USB_A, Connector_USB:USB_A_Molex_67643_Horizontal, symbol Connector:USB_A
- removed J6, J7: SD_Card_Receptacle, Connector_Card:SD_Card_Device_16mm_SlotDepth, symbol Connector:SD_Card_Receptacle
- removed U1: AMS1117CD-3.3, Package_TO_SOT_SMD:TO-252-3_TabPin2, symbol Regulator_Linear:AMS1117CD-3.3
- removed Y1: Crystal, Crystal:Crystal_SMD_3225-4Pin_3.2x2.5mm_HandSoldering, symbol Device:Crystal
- added GL850G2: GL850G, GL850G:28SSOP, symbol GL850G:GL850G
- added IC3, IC4: GL823K, GL823K:SOP64P600X175-16N, symbol GL823K:GL823K
- added J1, J3: USB_A, symbol Connector:USB_A
- added J2, J5: SD_Card_Receptacle, Connector_Card:SD_Kyocera_145638009511859+, symbol Connector:SD_Card_Receptacle
- added J4: USB_C_Receptacle_USB2.0_14P, symbol Connector:USB_C_Receptacle_USB2.0_14P
- R5: value 100kohm -> 100k
- R6: value 100kR -> 100k
Connections:
- net +3.3V: now also GL850G2.1 (AVDD@1), GL850G2.10 (AVDD@3), GL850G2.16 (DVDD), GL850G2.24 (3V3), GL850G2.5 (AVDD@2)
- net +3V3: now also J2.4 (VDD), J5.4 (VDD)
- net GND: now also R10.1, R7.2, R8.2, R9.1, GL850G2.14 (TEST), GL850G2.15 (GND), IC3.1 (VSS_1), IC3.14 (VSS_2), IC4.1 (VSS_1), IC4.14 (VSS_2), J1.4 (GND), J1.SH (Shield), J2.11 (WRITE_PROTECT), J2.3 (VSS), J2.6 (VSS), J2.SH (SHELL), J3.4 (GND), J3.SH (Shield), J4.A1 (GND), J4.A12 (GND), J4.B1 (GND), J4.B12 (GND), J4.SH (SHIELD), J5.11 (WRITE_PROTECT), J5.3 (VSS), J5.6 (VSS), J5.SH (SHELL); no longer D1.1 (K), D2.1 (K), R10.2, R9.2
- net SD1_CLK: now also IC3.4 (CLK), J5.5 (CLK)
- net SD1_CMD: now also IC3.5 (CMD), J5.2 (CMD)
- net SD1_D0: now also IC3.3 (D0), J5.7 (DAT0)
- net SD1_D1: now also IC3.2 (D1), J5.8 (DAT1)
- net SD1_D2: now also IC3.7 (D2), J5.9 (DAT2)
- net SD1_D3: now also IC3.6 (D3), J5.1 (CD/DAT3)
- net SD1_DM: now also GL850G2.27 (DM1), IC3.16 (DM)
- net SD1_DP: now also GL850G2.28 (DP1), IC3.15 (DP)
- net SD2_CLK: now also IC4.4 (CLK), J2.5 (CLK)
- net SD2_CMD: now also IC4.5 (CMD), J2.2 (CMD)
- net SD2_D0: now also IC4.3 (D0), J2.7 (DAT0)
- net SD2_D1: now also IC4.2 (D1), J2.8 (DAT1)
- net SD2_D2: now also IC4.7 (D2), J2.9 (DAT2)
- net SD2_D3: now also IC4.6 (D3), J2.1 (CD/DAT3)
- net SD2_DM: now also GL850G2.2 (DM2), IC4.16 (DM)
- net SD2_DP: now also GL850G2.3 (DP2), IC4.15 (DP)
- net USBA1_DM: now also GL850G2.8 (DM3), J1.2 (D-)
- net USBA1_DP: now also GL850G2.9 (DP3), J1.3 (D+)
- net USBA2_DM: now also GL850G2.11 (DM4), J3.2 (D-)
- net USBA2_DP: now also GL850G2.12 (DP4), J3.3 (D+)
- net USB_DM: now also GL850G2.25 (DM0), J4.A7 (D-), J4.B7 (D-)
- net USB_DP: now also GL850G2.26 (DP0), J4.A6 (D+), J4.B6 (D+)
- net VBUS: now also GL850G2.23 (5V), IC3.10 (5V), IC4.10 (5V), J1.1 (VBUS), J3.1 (VBUS), J4.A4 (VBUS), J4.A9 (VBUS), J4.B4 (VBUS), J4.B9 (VBUS)
- net at R6.1: now also GL850G2.19 (~{OVCUR2})
- net at R4.1: now also GL850G2.4 (RREF)
- net at D1.2 (A): now also D1.1 (K), R7.1, IC3.12 (LED); no longer R7.2
- net at R3.1: now also GL850G2.13 (~{RESET})
- net at R1.1: now also GL850G2.17 (PSELF)
- net at R2.1: now also GL850G2.18 (PGANG)
- net at R5.1: now also GL850G2.21 (~{OVCUR1})
- net at C12.1, C14.1: now also IC3.13 (VDDA), IC3.9 (VDD)
- net at C16.1, C17.1: now also IC4.13 (VDDA), IC4.9 (VDD)
- net at R8.1: now also D2.1 (K), D2.2 (A), IC4.12 (LED)
- new net: J4.A5 (CC1), R10.2
- new net: J4.B5 (CC2), R9.2
- no-connect marks 6 -> 10
Other:
- note removed: "GO DOWN ⬇︎ FOR SD CARD STUFF!!! SORRY!!! I RAN OUT OF SPACE"
- note removed: "are these NC or gnd </3"
- note removed: "pwr flag cuz kicad mad if i dont"
- moved on the sheet: C12, C14, C15, C16, C17, C19, C4, C5, C6, C7, C8, C9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

Commit message: yayyy done schema
:P
Parts:
- removed R3: 10kR, Resistor_SMD:R_0805_2012Metric, symbol Device:R
- added C1, C2: 22pF, Capacitor_SMD:C_0805_2012Metric, symbol Device:C
- added C10: 4.7uF, Capacitor_SMD:C_0805_2012Metric, symbol Device:C
- added C11, C20: 100nF, Capacitor_SMD:C_0805_2012Metric, symbol Device:C
- added C3: 1uF, Capacitor_SMD:C_0805_2012Metric, symbol Device:C
- added SW1: SW_Push, Button_Switch_SMD:SW_Push_SPST_NO_Alps_SKRK, symbol Switch:SW_Push
- added TP1, TP2, TP3, TP4: TestPoint, TestPoint:TestPoint_Pad_D1.0mm, symbol Connector:TestPoint
- added U2: SRV05-4, Package_TO_SOT_SMD:SOT-23-6, symbol Power_Protection:SRV05-4
- added Y1: 12MHz, Crystal:Crystal_SMD_3225-4Pin_3.2x2.5mm_HandSoldering, symbol Device:Crystal
- GL850G2: footprint GL850G:28SSOP -> GL850G Model:28SSOP
- IC3, IC4: footprint GL823K:SOP64P600X175-16N -> GL823K Model by Genesys Logic:SOP64P600X175-16N
- J1, J3: footprint (none) -> Connector_USB:USB_A_Connfly_DS1098_Horizontal
- J4: footprint (none) -> Connector_USB:USB_C_Receptacle_HRO_TYPE-C-31-M-12
- renumbered U2 to U1
Connections:
- net +3.3V: now also TP4.1
- net +3V3: no longer J2.4 (VDD), J5.4 (VDD)
- net GND: now also C13.2, C15.2, IC3.10 (5V), IC4.10 (5V), C1.1, C10.1, C11.2, C2.2, C20.2, C3.1, SW1.1, TP2.1, U2.2 (VN); no longer C13.1, C15.1
- net SD2_CLK: now also IC4.5 (CMD); no longer IC4.4 (CLK)
- net SD2_CMD: now also IC4.4 (CLK), R16.2; no longer IC4.5 (CMD), R20.2
- net SD2_D0: now also IC4.6 (D3), R20.2; no longer IC4.3 (D0), R16.2
- net SD2_D1: now also IC4.7 (D2), R19.2; no longer IC4.2 (D1), R17.2
- net SD2_D2: now also IC4.2 (D1); no longer IC4.7 (D2)
- net SD2_D3: now also IC4.3 (D0), R17.2; no longer IC4.6 (D3), R19.2
- net USBA1_DM: now also U2.3 (IO2)
- net USBA1_DP: now also U2.1 (IO1)
- net USBA2_DM: now also U2.6 (IO4)
- net USBA2_DP: now also U2.4 (IO3)
- net VBUS: now also C13.1, C15.1, C10.2, C11.1, C20.1, TP1.1, U2.5 (VP); no longer C13.2, C15.2, IC3.10 (5V), IC4.10 (5V)
- net at D2.2 (A), IC4.12 (LED): no longer D2.1 (K), R8.1
- net at IC4.8 (PMOS): now also J2.4 (VDD)
- net at GL850G2.13 (~{RESET}): now also C3.2, SW1.2, TP3.1
- net at GL850G2.6 (X1): now also C1.2, Y1.2
- net at GL850G2.7 (X2): now also C2.1, Y1.1
- net at D1.2 (A), IC3.12 (LED): no longer D1.1 (K), R7.1
- net at IC3.8 (PMOS): now also J5.4 (VDD)
- new net: D1.1 (K), R7.1
- new net: D2.1 (K), R8.1
- no-connect marks 10 -> 6
Other:
- moved on the sheet: C12, C13, C14, C16, C17, C19, C4, C5, C6, C7, C8, C9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

Commit message: give up on schematic
im tired i need sleep
Changed lines of the file:
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@@
 	)
 	(junction
+		(at 238.76 203.2)
+		(diameter 0)
+		(color 0 0 0 0)
+	)
+	(junction
 		(at 73.66 41.91)
 		(diameter 0)
@@
 	)
 	(junction
+		(at 347.98 199.39)
+		(diameter 0)
+		(color 0 0 0 0)
+	)
+	(junction
 		(at 35.56 77.47)
 		(diameter 0)
@@
 	(wire
 		(pts
-			(xy 347.98 204.47) (xy 347.98 175.26)
+			(xy 347.98 204.47) (xy 347.98 199.39)
 		)
 		(stroke
@@
 	(wire
 		(pts
-			(xy 187.96 109.22) (xy 190.5 109.22)
+			(xy 176.53 109.22) (xy 190.5 109.22)
 		)
 		(stroke
@@
 	(wire
 		(pts
+			(xy 259.08 219.71) (xy 254 219.71)
+		)
+		(stroke
+			(width 0)
+			(type default)
+		)
+	)
+	(wire
+		(pts
 			(xy 172.72 104.14) (xy 172.72 101.6)
 		)
@@
 	(wire
 		(pts
+			(xy 347.98 199.39) (xy 347.98 175.26)
+		)
+		(stroke
+			(width 0)
+			(type default)
+		)
+	)
+	(wire
+		(pts
 			(xy 318.77 165.1) (xy 328.93 165.1)
 		)
@@
 	(wire
 		(pts
-			(xy 369.57 217.17) (xy 363.22 217.17)
+			(xy 363.22 217.17) (xy 369.57 217.17)
 		)
 		(stroke
@@
 	(wire
 		(pts
+			(xy 238.76 203.2) (xy 238.76 207.01)
+		)
+		(stroke
+			(width 0)
+			(type default)
+		)
+	)
+	(wire
+		(pts
 			(xy 77.47 49.53) (xy 77.47 44.45)
 		)
@@
 	(wire
 		(pts
-			(xy 238.76 175.26) (xy 238.76 207.01)
+			(xy 238.76 175.26) (xy 238.76 203.2)
 		)
 		(stroke
@@
 		(dnp no)
 		(property "Reference" "D1"
-			(at 262.89 163.576 0)
+			(at 263.906 164.846 0)
 			(show_name no)
 			(do_not_autoplace no)
@@
 	)
 	(symbol
+		(lib_id "power:PWR_FLAG")
+		(at 238.76 203.2 90)
+		(unit 1)
+		(body_style 1)
+		(exclude_from_sim no)
+		(in_bom yes)
+		(on_board yes)
+		(in_pos_files yes)
+		(dnp no)
+		(fields_autoplaced yes)
+		(property "Reference" "#FLG04"
+			(at 236.855 203.2 0)
+			(hide yes)
+			(show_name no)
+			(do_not_autoplace no)
+			(effects
+				(font
+					(size 1.27 1.27)
+				)
+			)
+		)
+		(property "Value" "PWR_FLAG"
+			(at 234.95 203.1999 90)
+			(show_name no)
+			(do_not_autoplace no)
+			(effects
+				(font
+					(size 1.27 1.27)
+				)
+				(justify left)
+			)
+		)
+		(property "Footprint" ""
+			(at 238.76 203.2 0)
+			(hide yes)
+			(show_name no)
+			(do_not_autoplace no)
+			(effects
+				(font
+					(size 1.27 1.27)
+				)
+			)
+		)
+		(property "Datasheet" ""
+			(at 238.76 203.2 0)
+			(hide yes)
+			(show_name no)
+			(do_not_autoplace no)
+			(effects
+				(font
+					(size 1.27 1.27)
+				)
+			)
+		)
+		(property "Description" "Special symbol for telling ERC where power comes from"
+			(at 238.76 203.2 0)
+			(hide yes)
+			(show_name no)
+			(do_not_autoplace no)
+			(effects
+				(font
+					(size 1.27 1.27)
+				)
+			)
+		)
+		(pin "1"
+		)
+		(instances
+			(project "a-side"
+				(path "/4689210d-3702-4f71-a790-ad3b060da840"
+					(reference "#FLG04")
+					(unit 1)
+				)
+			)
+		)
+	)
+	(symbol
 		(lib_id "Device:R")
 		(at 302.26 194.31 0)
@@
 	)
 	(symbol
+		(lib_id "power:PWR_FLAG")
+		(at 347.98 199.39 270)
+		(unit 1)
+		(body_style 1)
+		(exclude_from_sim no)
+		(in_bom yes)
+		(on_board yes)
+		(in_pos_files yes)
+		(dnp no)
+		(fields_autoplaced yes)
+		(property "Reference" "#FLG05"
+			(at 349.885 199.39 0)
+			(hide yes)
+			(show_name no)
+			(do_not_autoplace no)
+			(effects
+				(font
+					(size 1.27 1.27)
+				)
+			)
+		)
+		(property "Value" "PWR_FLAG"
+			(at 351.79 199.3899 90)
+			(show_name no)
+			(do_not_autoplace no)
+			(effects
+				(font
+					(size 1.27 1.27)
+				)
+				(justify left)
+			)
+		)
+		(property "Footprint" ""
+			(at 347.98 199.39 0)
+			(hide yes)
+			(show_name no)
+			(do_not_autoplace no)
+			(effects
+				(font
+					(size 1.27 1.27)
+				)
+			)
+		)
+		(property "Datasheet" ""
+			(at 347.98 199.39 0)
+			(hide yes)
+			(show_name no)
+			(do_not_autoplace no)
+			(effects
+				(font
+					(size 1.27 1.27)
+				)
+			)
+		)
+		(property "Description" "Special symbol for telling ERC where power comes from"
+			(at 347.98 199.39 0)
+			(hide yes)
+			(show_name no)
+			(do_not_autoplace no)
+			(effects
+				(font
+					(size 1.27 1.27)
+				)
+			)
+		)
+		(pin "1"
+		)
+		(instances
+			(project "a-side"
+				(path "/4689210d-3702-4f71-a790-ad3b060da840"
+					(reference "#FLG05")
+					(unit 1)
+				)
+			)
+		)
+	)
+	(symbol
 		(lib_id "power:GND")
 		(at 73.66 238.76 0)
@@
 	(symbol
 		(lib_id "power:GND")
-		(at 254 219.71 0)
+		(at 259.08 219.71 0)
 		(unit 1)
 		(body_style 1)
@@
 		(fields_autoplaced yes)
 		(property "Reference" "#PWR03"
-			(at 254 226.06 0)
+			(at 259.08 226.06 0)
 			(hide yes)
 			(show_name no)
@@
 		)
 		(property "Value" "GND"
-			(at 254 224.79 0)
+			(at 259.08 224.79 0)
 			(show_name no)
 			(do_not_autoplace no)
@@
 		)
 		(property "Footprint" ""
-			(at 254 219.71 0)
+			(at 259.08 219.71 0)
 			(hide yes)
 			(show_name no)
@@
 		)
 		(property "Datasheet" ""
-			(at 254 219.71 0)
+			(at 259.08 219.71 0)
 			(hide yes)
 			(show_name no)
@@
 		)
 		(property "Description" "Power symbol creates a global label with name \"GND\" , ground"
-			(at 254 219.71 0)
+			(at 259.08 219.71 0)
 			(hide yes)
 			(show_name no)
@@
 	(symbol
 		(lib_id "power:GND")
-		(at 187.96 109.22 0)
+		(at 176.53 109.22 0)
 		(unit 1)
 		(body_style 1)
@@
 		(fields_autoplaced yes)
 		(property "Reference" "#PWR022"
-			(at 187.96 115.57 0)
+			(at 176.53 115.57 0)
 			(hide yes)
 			(show_name no)
@@
 		)
 		(property "Value" "GND"
-			(at 187.96 114.3 0)
+			(at 176.53 114.3 0)
 			(show_name no)
 			(do_not_autoplace no)
@@
 		)
 		(property "Footprint" ""
-			(at 187.96 109.22 0)
+			(at 176.53 109.22 0)
 			(hide yes)
 			(show_name no)
@@
 		)
 		(property "Datasheet" ""
-			(at 187.96 109.22 0)
+			(at 176.53 109.22 0)
 			(hide yes)
 			(show_name no)
@@
 		)
 		(property "Description" "Power symbol creates a global label with name \"GND\" , ground"
-			(at 187.96 109.22 0)
+			(at 176.53 109.22 0)
 			(hide yes)
 			(show_name no)
