File: a-side/_autosave-a-side.kicad_pcb (KiCad board)
At the start: 2 copper layers, 95 x 55 mm, 40 parts, among them IC1 GL823K, IC2 GL823K, J2 USB_C_Receptacle_USB2.0_14P, J4 USB_A, J5 USB_A, U1 AMS1117CD-3.3, U2 SRV05-4, Y1 Crystal

Commit message: work !!
fixingmostly schematic and stuff yay still working
Connections:
- C18 pad 1: GND -> +3.3V
- C18 pad 2: +3.3V -> GND
- C3 pad 1: VBUS -> GND
- C3 pad 2: GND -> VBUS
- D1 pad 1: Net-(D1-K) -> GND
- D1 pad 2: GND -> Net-(D1-A)
- D2 pad 1: Net-(D2-K) -> GND
- D2 pad 2: GND -> Net-(D2-A)
- R7 pad 2: Net-(D1-K) -> Net-(D1-A)
- R8 pad 2: Net-(D2-K) -> Net-(D2-A)
Changed lines of the file:
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@@
 	(net 6 "Net-(IC1-VDD)")
 	(net 7 "Net-(IC2-VDD)")
-	(net 8 "Net-(D1-K)")
-	(net 9 "Net-(D2-K)")
+	(net 8 "Net-(D1-A)")
+	(net 9 "Net-(D2-A)")
 	(net 10 "/SD1_DM")
 	(net 11 "unconnected-(GL850G1-PWREN2-Pad20)")
@@
 			(layers "F.Cu" "F.Mask" "F.Paste")
 			(roundrect_rratio 0.25)
-			(net 2 "GND")
+			(net 3 "+3.3V")
 			(pintype "passive")
 		)
@@
 			(layers "F.Cu" "F.Mask" "F.Paste")
 			(roundrect_rratio 0.25)
-			(net 3 "+3.3V")
+			(net 2 "GND")
 			(pintype "passive")
 		)
@@
 			(layers "F.Cu" "F.Mask" "F.Paste")
 			(roundrect_rratio 0.217391)
-			(net 8 "Net-(D1-K)")
+			(net 2 "GND")
 			(pinfunction "K")
 			(pintype "passive")
@@
 			(layers "F.Cu" "F.Mask" "F.Paste")
 			(roundrect_rratio 0.217391)
-			(net 2 "GND")
+			(net 8 "Net-(D1-A)")
 			(pinfunction "A")
 			(pintype "passive")
@@
 			(layers "F.Cu" "F.Mask" "F.Paste")
 			(roundrect_rratio 0.243902)
-			(net 9 "Net-(D2-K)")
+			(net 9 "Net-(D2-A)")
 			(pintype "passive")
 		)
@@
 			(layers "F.Cu" "F.Mask" "F.Paste")
 			(roundrect_rratio 0.243902)
-			(net 8 "Net-(D1-K)")
+			(net 8 "Net-(D1-A)")
 			(pintype "passive")
 		)
@@
 			(layers "F.Cu" "F.Mask" "F.Paste")
 			(roundrect_rratio 0.217391)
-			(net 9 "Net-(D2-K)")
+			(net 2 "GND")
 			(pinfunction "K")
 			(pintype "passive")
@@
 			(layers "F.Cu" "F.Mask" "F.Paste")
 			(roundrect_rratio 0.217391)
-			(net 2 "GND")
+			(net 9 "Net-(D2-A)")
 			(pinfunction "A")
 			(pintype "passive")
@@
 			(layers "F.Cu" "F.Mask" "F.Paste")
 			(roundrect_rratio 0.25)
-			(net 1 "VBUS")
+			(net 2 "GND")
 			(pintype "passive")
 		)
@@
 			(layers "F.Cu" "F.Mask" "F.Paste")
 			(roundrect_rratio 0.25)
-			(net 2 "GND")
+			(net 1 "VBUS")
 			(pintype "passive")
 		)
