File: a-side/_autosave-a-side.kicad_sch (KiCad schematic)
At the start: 52 parts, among them IC1 GL823K, IC2 GL823K, J2 USB_C_Receptacle_USB2.0_14P, J4 USB_A, J5 USB_A, J6 SD_Card_Receptacle, J7 SD_Card_Receptacle, U1 AMS1117CD-3.3, U2 SRV05-4, Y1 Crystal

Commit message: work !!
fixingmostly schematic and stuff yay still working
Connections:
- net GND: now also J6.10 (CARD_DETECT), J6.11 (WRITE_PROTECT), J6.12 (SHELL1), J6.13 (SHELL2), J7.10 (CARD_DETECT), J7.11 (WRITE_PROTECT), J7.12 (SHELL1), J7.13 (SHELL2)
- no-connect marks 14 -> 6
